File: experiments/hardwareddc-aux-breakout/hardwareddc-aux-breakout.kicad_pcb (KiCad board)
At the start: 4 copper layers, 54.3 x 75 mm, 19 parts, among them J1 Conn_01x04_Pin, J2 USB_C_Receptacle, J3 Conn_01x03_Pin, J4 Conn_01x02_Pin, J5 472720001, J6 472720001, J7 HDMI_A_1.4, U1 SN65MLVD200ADR, U2 AMS1117-3.3

Commit message: update experiment: HardwareDDC Aux V2.0
Parts:
- C1: footprint Capacitor_SMD:C_01005_0402Metric -> Capacitor_SMD:C_0402_1005Metric
- R1, R2: footprint Resistor_SMD:R_01005_0402Metric -> Resistor_SMD:R_0402_1005Metric
- moved C1 1.26 mm to (142.8, 80.6)
- moved R1 0.51 mm to (143.6, 81.8)
- moved R2 0.51 mm to (143.6, 79.3)
Routing:
- net GND: track 70.5 -> 72.1 mm, vias 43 -> 42
- net +5V: track 26.4 -> 27.5 mm
- net /SDA: vias 5 -> 4
